File: Lestanarve_hw/Lestanarve.kicad_sch (KiCad schematic)
At the start: 51 parts

Commit message: + UART works
Parts:
- removed C?: 10u, Capacitors:CAP_0603, symbol Tittar_kl:C
- removed L?: BLM15AG102SN1, Inductors:IND_0402, symbol Tittar_kl:L
- removed Logo?: Logo, Pictures:Ostranna_16d9_13d5, symbol pcb_details:Logo
- removed R?: 4k7, Resistors:RES_0603, symbol Tittar_kl:R
- removed SW?: BUTTON, BtnsSwitches:BTN_4x4_SMD, symbol Switches:BUTTON
- added R6: 1k2, Resistors:RES_0603, symbol Tittar_kl:R
- added SW1: SWITCH, BtnsSwitches:SW_SS-1P2T_Housing, symbol BtnsSwitches:SWITCH_1P2T_housing
- added XL3: CONN_6, Connectors:PLS-6-NoHole, symbol Connectors_kl:CONN_6
- C1, C10, C11, C12, C15, C16, C17, C18, C2, C3, C4, C5, C6, C7, C8, C9: renamed from C?; footprint Capacitors:CAP_0603 -> Capacitors:CAP_0603_Silks
- D1: renamed from D?; footprint LEDs:LED_0603 -> LEDs:LED_0603_ch
- D2: renamed from D?; Price 2 -> 5
- L1: renamed from L?; PN (none) -> -; Price (none) -> 4; SolderPoints (none) -> 2; Tolerance (none) -> 20%; Type (none) -> Inductor SMD
- XL1: renamed from XL?; footprint Connectors:PLS-6-NoHole -> Connectors:PLS-6_LOCK
- gave numbers to parts that had none: 26
Connections:
- net BLUE_LED is gone; now on net UART_RX: DD2.31 (T1C3/SDA1/SAI1SDA/RX1/PA10)
- net GREEN_LED is gone; now on net UART_TX: DD2.30 (T1C2/SCL1/SAI1FSA/TX1/PA9)
- net IR_LEVEL is gone; now on net CC_GDO0: DD2.14 (ADC9/SAI1FSB/LPTIM2_OUT/DAC1/CK2/PA4)
- net LUMOS_CTRL is gone; now on net CC_MISO: DD2.16 (ADC11/T16C1/MISO1/PA6)
- net PwrMCU is gone; now on net +3v3: C10.1, C6.2, C7.1, C8.1, C9.1, DD2.1 (VBAT), DD2.24 (VDD), DD2.36 (VDDUSB), DD2.48 (VDD), L1.1, XL1.1
- net +3v3: now also XL3.2
- net +BATT: now also SW1.1; no longer Q3.3 (D)
- net 5V_USB: no longer R2.2
- net ADC_BAT_EN: now also DD2.18 (PB0/T1C2N/CK3/SAI1EXTCLK/ADC15); no longer DD2.15 (ADC10/T2C1ETR/DAC2/SCK1/PA5)
- net CC_GDO0: now also XL3.6; no longer DD2.18 (PB0/T1C2N/CK3/SAI1EXTCLK/ADC15)
- net CC_MISO: now also XL3.4; no longer DD2.40 (PB4/MISO1/MISO3/SDA3/SAI1MCLKB)
- net CC_MOSI: now also DD2.17 (ADC12/T1C1N/SCL3/MOSI1/PA7), XL3.3; no longer DD2.41 (PB5/MOSI1/MOSI3/CK1/LPTIM1_IN1/SAI1SDB)
- net CC_SCK: now also DD2.15 (ADC10/T2C1ETR/DAC2/SCK1/PA5), XL3.5; no longer DD2.39 (PB3/SCK1/SCK3/T2C2/SWO/SAI1SCKB)
- net GND: now also D1.C, R6.2, SW1.H, XL3.1
- net IS_CHARGING: now also DD2.10 (ADC5/WKUP1/T2C1ETR/PA0); no longer D1.C, DD2.12 (ADC7/WKUP4/T15C1/T2C3/LP1TX/TX2/PA2)
- net NPX1_CTRL: now also DD2.41 (PB5/MOSI1/MOSI3/CK1/LPTIM1_IN1/SAI1SDB)
- net NPX_PWR_EN: now also DD2.42 (PB6/SCL1/T16C1N/TX1/SAI1FSB)
- net UART_RX: no longer DD2.43 (PB7/SDA1/RX1/LPTIM1_IN2)
- net UART_TX: no longer DD2.42 (PB6/SCL1/T16C1N/TX1/SAI1FSB)
- net at R1.1: now also DD2.12 (ADC7/WKUP4/T15C1/T2C3/LP1TX/TX2/PA2)
- net at DA2.2 (PROG): now also R6.1
- net CC_CS: no longer names the net of DD2.38 (T2C1ETR/RX2/PA15)
- net EE_PWR: no longer names the net of DD2.21 (PB10/T2C3/SCK2/SCL2/TX3/LPRX1/SAI1SCKA)
- net IR_CARRIER: no longer names the net of DD2.20 (PB2/LPTIM1_OUT/RTC_OUT)
- net PwrUnst renamed +PwrUnst
- net RED_LED: no longer names the net of DD2.29 (LPTIM2_OUT/MCO/T1C1/CK1/SAI1SCKA/PA8)
- net SCL: no longer names the net of DD2.45 (PB8/SDIO_D4/T16C1/SCL1/SAI1MCLKA)
- net SCL: now also R2.2
- net SDA: no longer names the net of DD2.46 (PB9/SDIO_D5/SDA1/IR_OUT/SAI1FSA)
- net VIBRO_CTRL: no longer names the net of DD2.13 (ADC8/SAI1MCLKA/T15C2/T2C4/LP1RX/RX2/PA3)
- new net: Q3.3 (D), SW1.2
- no-connect marks 10 -> 19
Other:
- note added: "Charger 1.2k => 1000mA"
- note added: "MOSI3"
- note removed: "Charger 4k7 => 270 mA"
- note removed: "DAC1"
- note removed: "I2C1"
- note removed: "LPTIM1 OUT OpenDrain"
- note removed: "T15C2"
- note removed: "T1C1"
- note removed: "T1C2"
- note removed: "T1C3"
- moved on the sheet: C13, C17, C18, D1, D2, DA1, DA3, Q1, Q2, Q3, R1, R11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
